Commit message: fix box size: not to zero

File: kinova_description/urdf/j2n6s300_standalone.xacro (robot description, xacro)
@@ -19,5 +19,5 @@
       <origin xyz="0 0 0" rpy="0 0 0" />
       <geometry>
-        <box size = "0 0 0"/>
+        <box size = "0.00001 0.00001 0.00001"/>
       </geometry>
     <!--<material name="Black" /> -->
@@ -26,5 +26,5 @@
       <origin xyz="0 0 0" rpy="0 0 0" />
       <geometry>
-        <box size = "0 0 0"/>
+        <box size = "0.00001 0.00001 0.00001"/>
       </geometry>
     </collision>

File: kinova_description/urdf/kinova_common.xacro (robot description, xacro)
@@ -70,10 +70,10 @@
             <visual>
                 <geometry>
-                    <box size = "0 0 0"/>
+                    <box size = "0.00001 0.00001 0.00001"/>
                 </geometry>
             </visual>
             <collision>
                 <geometry>
-                    <box size = "0 0 0"/>
+                    <box size = "0.00001 0.00001 0.00001"/>
                 </geometry>
             </collision>
